File: parachute_ignition/parachute_ignition.sch (KiCad schematic (older format))
At the start: 9 parts, among them P1 CONN_01X02, Q1 IRF7456PBF, U1 LM555N, U2 74LS14

Commit message: ignition on for 860 ms
Parts:
- C1: value 100uF -> 470uF
- R1: value 1k -> 2k7
- RV1: value 33k -> 8k2
Changed lines of the file:
@@
 P 6150 3100
 F 0 "R1" V 6230 3100 40  0000 C CNN
-F 1 "1k" V 6157 3101 40  0000 C CNN
+F 1 "2k7" V 6157 3101 40  0000 C CNN
 F 2 "" V 6080 3100 30  0000 C CNN
 F 3 "" H 6150 3100 30  0000 C CNN
@@
 P 4450 3750
 F 0 "C1" H 4450 3850 40  0000 L CNN
-F 1 "100uF" H 4456 3665 40  0000 L CNN
+F 1 "470uF" H 4456 3665 40  0000 L CNN
 F 2 "" H 4488 3600 30  0000 C CNN
 F 3 "" H 4450 3750 60  0000 C CNN
@@
 P 5300 3500
 F 0 "RV1" H 5300 3400 50  0000 C CNN
-F 1 "33k" H 5300 3500 50  0000 C CNN
+F 1 "8k2" H 5300 3500 50  0000 C CNN
 F 2 "" H 5300 3500 60  0000 C CNN
 F 3 "" H 5300 3500 60  0000 C CNN
