File: parachute_ignition/parachute_ignition.sch (KiCad schematic (older format))
At the start: 9 parts, among them P1 CONN_01X02, Q1 IRF7413ZPBF, U1 4047

Commit message: last improvments and pcbs
Connections:
- wire segments 25 -> 31
Changed lines of the file:
@@
 $EndComp
 $Comp
+L VCC #PWR01
+U 1 1 5415C86E
+P 8000 3050
+F 0 "#PWR01" H 8000 3150 30  0001 C CNN
+F 1 "VCC" H 8000 3150 30  0000 C CNN
+F 2 "" H 8000 3050 60  0000 C CNN
+F 3 "" H 8000 3050 60  0000 C CNN
+	1    8000 3050
+	1    0    0    -1
+$EndComp
+$Comp
+L GND #PWR02
+U 1 1 5415C882
+P 8000 3750
+F 0 "#PWR02" H 8000 3750 30  0001 C CNN
+F 1 "GND" H 8000 3680 30  0001 C CNN
+F 2 "" H 8000 3750 60  0000 C CNN
+F 3 "" H 8000 3750 60  0000 C CNN
+	1    8000 3750
 	1    0    0    -1
 $EndComp
@@
 F 0 "Q1" H 6385 4035 40  0000 C CNN
 F 1 "IRF7413ZPBF" H 6550 3515 40  0000 C CNN
-F 2 "SMD_Packages:SOIC-8-W" H 6550 3950 30  0000 C CIN
+F 2 "SMD_Packages:SOIC-8-W" H 6550 3950 30  0001 C CIN
 F 3 "" V 6550 3750 60  0000 C CNN
 	1    6550 3750
@@
 $EndComp
 Wire Wire Line
-	7000 3550 6850 3550
+	6850 3550 7000 3550
 Wire Wire Line
 	6200 3750 6250 3750
@@
 Wire Wire Line
 	6950 3100 6900 3100
+Wire Wire Line
+	6250 3650 6200 3650
+Connection ~ 6200 3650
+Wire Wire Line
+	6250 3550 6200 3550
+Connection ~ 6200 3550
+Wire Wire Line
+	6850 3650 6900 3650
+Wire Wire Line
+	6900 3550 6900 3850
+Connection ~ 6900 3550
+Wire Wire Line
+	6900 3750 6850 3750
+Connection ~ 6900 3650
+Wire Wire Line
+	6900 3850 6850 3850
+Connection ~ 6900 3750
 $EndSCHEMATC
